Commit message: xmllint auto-formatting

File: fanuc_m10ia_ensenso/fanuc_m10ia_ensenso_support/urdf/m10ia_ensenso_eef.xacro (robot description, xacro)
@@ -1,4 +1,4 @@
-<?xml version="1.0" ?>
-<robot name="fanuc_m10ia_ensenso" xmlns:xacro="http://ros.org/wiki/xacro">
+<?xml version="1.0"?>
+<robot xmlns:xacro="http://ros.org/wiki/xacro" name="fanuc_m10ia_ensenso">
   <xacro:include filename="$(find fanuc_m10ia_ensenso_support)/urdf/m10ia_ensenso_eef_macro.xacro"/>
   <xacro:fanuc_m10ia_ensenso_support prefix=""/>

File: fanuc_m10ia_ensenso/fanuc_m10ia_ensenso_support/urdf/m10ia_ensenso_eef_macro.xacro (robot description, xacro)
@@ -4,30 +4,30 @@
   <xacro:include filename="$(find fanuc_m10ia_support)/urdf/m10ia_macro.xacro"/>
   <xacro:include filename="$(find fanuc_m10ia_ensenso_support)/urdf/mounting_plate_macro.xacro"/>
-  <xacro:include filename="$(find ensenso_n10_description)/urdf/ensenso_n10_macro.xacro" />
+  <xacro:include filename="$(find ensenso_n10_description)/urdf/ensenso_n10_macro.xacro"/>
   <!-- create the robot and eef combo itself as a macro -->
   <xacro:macro name="fanuc_m10ia_ensenso_support" params="prefix">
-  <!-- instantiate everything -->
-  <xacro:fanuc_m10ia prefix="${prefix}" />
-  <xacro:mounting_plate prefix="${prefix}" />
-  <xacro:ensenso_n10 prefix="${prefix}" />
-  <!-- attach mounting plate to M-10iA model -->
-  <joint name="${prefix}tool0-mounting_plate_base_link" type="fixed">
-    <origin xyz="0 0 0.008" rpy="0 0 0" />
-    <parent link="${prefix}tool0" />
-    <child link="${prefix}mounting_plate_base_link" />
-  </joint>
-  <!-- attach eef to robot model -->
-  <joint name="${prefix}tool0-ensenso_n10_frame" type="fixed">
-    <origin xyz="0 -0.088 0.032" rpy="0 0 -1.5707" />
-    <parent link="${prefix}tool0" />
-    <child link="${prefix}ensenso_n10_frame" />
-  </joint>
-  <link name="${prefix}ensenso_tcp">
+    <!-- instantiate everything -->
+    <xacro:fanuc_m10ia prefix="${prefix}"/>
+    <xacro:mounting_plate prefix="${prefix}"/>
+    <xacro:ensenso_n10 prefix="${prefix}"/>
+    <!-- attach mounting plate to M-10iA model -->
+    <joint name="${prefix}tool0-mounting_plate_base_link" type="fixed">
+      <origin xyz="0 0 0.008" rpy="0 0 0"/>
+      <parent link="${prefix}tool0"/>
+      <child link="${prefix}mounting_plate_base_link"/>
+    </joint>
+    <!-- attach eef to robot model -->
+    <joint name="${prefix}tool0-ensenso_n10_frame" type="fixed">
+      <origin xyz="0 -0.088 0.032" rpy="0 0 -1.5707"/>
+      <parent link="${prefix}tool0"/>
+      <child link="${prefix}ensenso_n10_frame"/>
+    </joint>
+    <link name="${prefix}ensenso_tcp">
   </link>
-  <joint name="${prefix}tool0-ensenso_tcp_frame" type="fixed">
-    <origin xyz="0 -0.088 0.035" rpy="0 0 -1.5707" />
-    <parent link="${prefix}tool0" />
-    <child link="${prefix}ensenso_tcp" />
-  </joint>
+    <joint name="${prefix}tool0-ensenso_tcp_frame" type="fixed">
+      <origin xyz="0 -0.088 0.035" rpy="0 0 -1.5707"/>
+      <parent link="${prefix}tool0"/>
+      <child link="${prefix}ensenso_tcp"/>
+    </joint>
   </xacro:macro>
 </robot>

File: fanuc_m10ia_ensenso/fanuc_m10ia_ensenso_support/urdf/mounting_plate.xacro (robot description, xacro)
@@ -1,4 +1,4 @@
-<?xml version="1.0" ?>
-<robot name="mounting_plate" xmlns:xacro="http://ros.org/wiki/xacro">
+<?xml version="1.0"?>
+<robot xmlns:xacro="http://ros.org/wiki/xacro" name="mounting_plate">
   <xacro:include filename="$(find fanuc_m10ia_ensenso_support)/urdf/mounting_plate_macro.xacro"/>
   <xacro:mounting_plate prefix=""/>

File: fanuc_m10ia_kinect/fanuc_m10ia_kinect_support/urdf/m10ia_kinect_eef.xacro (robot description, xacro)
@@ -1,4 +1,4 @@
-<?xml version="1.0" ?>
-<robot name="fanuc_m10ia_kinect" xmlns:xacro="http://ros.org/wiki/xacro">
+<?xml version="1.0"?>
+<robot xmlns:xacro="http://ros.org/wiki/xacro" name="fanuc_m10ia_kinect">
   <xacro:include filename="$(find fanuc_m10ia_kinect_support)/urdf/m10ia_kinect_eef_macro.xacro"/>
   <xacro:fanuc_m10ia_kinect_support prefix=""/>

File: fanuc_m10ia_kinect/fanuc_m10ia_kinect_support/urdf/m10ia_kinect_eef_macro.xacro (robot description, xacro)
@@ -4,30 +4,30 @@
   <xacro:include filename="$(find fanuc_m10ia_support)/urdf/m10ia_macro.xacro"/>
   <xacro:include filename="$(find fanuc_m10ia_kinect_support)/urdf/mounting_plate_macro.xacro"/>
-  <xacro:include filename="$(find kinect_v1_description)/urdf/kinect_v1_macro.xacro" />
+  <xacro:include filename="$(find kinect_v1_description)/urdf/kinect_v1_macro.xacro"/>
   <!-- create the robot and eef combo itself as a macro -->
   <xacro:macro name="fanuc_m10ia_kinect_support" params="prefix">
-  <!-- instantiate everything -->
-  <xacro:fanuc_m10ia prefix="${prefix}" />
-  <xacro:mounting_plate prefix="${prefix}" />
-  <xacro:kinect_v1 prefix="${prefix}" />
-  <!-- attach mounting plate to M-10iA model -->
-  <joint name="${prefix}tool0-mounting_plate_base_link" type="fixed">
-    <origin xyz="0 0 0.008" rpy="0 0 0" />
-    <parent link="${prefix}tool0" />
-    <child link="${prefix}mounting_plate_base_link" />
-  </joint>
-  <!-- attach eef to robot model -->
-  <joint name="${prefix}tool0-kinect_v1_frame" type="fixed">
-    <origin xyz="0 -0.01 0.028" rpy="0 0 0" />
-    <parent link="${prefix}tool0" />
-    <child link="${prefix}kinect_v1_frame" />
-  </joint>
-  <link name="${prefix}kinect_tcp">
+    <!-- instantiate everything -->
+    <xacro:fanuc_m10ia prefix="${prefix}"/>
+    <xacro:mounting_plate prefix="${prefix}"/>
+    <xacro:kinect_v1 prefix="${prefix}"/>
+    <!-- attach mounting plate to M-10iA model -->
+    <joint name="${prefix}tool0-mounting_plate_base_link" type="fixed">
+      <origin xyz="0 0 0.008" rpy="0 0 0"/>
+      <parent link="${prefix}tool0"/>
+      <child link="${prefix}mounting_plate_base_link"/>
+    </joint>
+    <!-- attach eef to robot model -->
+    <joint name="${prefix}tool0-kinect_v1_frame" type="fixed">
+      <origin xyz="0 -0.01 0.028" rpy="0 0 0"/>
+      <parent link="${prefix}tool0"/>
+      <child link="${prefix}kinect_v1_frame"/>
+    </joint>
+    <link name="${prefix}kinect_tcp">
   </link>
-  <joint name="${prefix}tool0-kinect_tcp_frame" type="fixed">
-    <origin xyz="0 -0.01 0.028" rpy="0 0 0" />
-    <parent link="${prefix}tool0" />
-    <child link="${prefix}kinect_tcp" />
-  </joint>
+    <joint name="${prefix}tool0-kinect_tcp_frame" type="fixed">
+      <origin xyz="0 -0.01 0.028" rpy="0 0 0"/>
+      <parent link="${prefix}tool0"/>
+      <child link="${prefix}kinect_tcp"/>
+    </joint>
   </xacro:macro>
 </robot>

File: fanuc_m10ia_kinect/fanuc_m10ia_kinect_support/urdf/mounting_plate.xacro (robot description, xacro)
@@ -1,4 +1,4 @@
-<?xml version="1.0" ?>
-<robot name="mounting_plate" xmlns:xacro="http://ros.org/wiki/xacro">
+<?xml version="1.0"?>
+<robot xmlns:xacro="http://ros.org/wiki/xacro" name="mounting_plate">
   <xacro:include filename="$(find fanuc_m10ia_kinect_support)/urdf/mounting_plate_macro.xacro"/>
   <xacro:mounting_plate prefix=""/>

File: fanuc_r1000ia_grinding/fanuc_r1000ia_ensenso_n10_grinding_support/urdf/r1000ia_grinding.xacro (robot description, xacro)
@@ -1,4 +1,4 @@
-<?xml version="1.0" ?>
-<robot name="fanuc_r1000ia_grinding" xmlns:xacro="http://ros.org/wiki/xacro">
+<?xml version="1.0"?>
+<robot xmlns:xacro="http://ros.org/wiki/xacro" name="fanuc_r1000ia_grinding">
   <xacro:include filename="$(find fanuc_r1000ia_ensenso_n10_grinding_support)/urdf/r1000ia_grinding_macro.xacro"/>
   <xacro:fanuc_r1000ia_ensenso_n10_grinding_support prefix=""/>

File: fanuc_r1000ia_grinding/fanuc_r1000ia_ensenso_n10_grinding_support/urdf/r1000ia_grinding_macro.xacro (robot description, xacro)
@@ -3,46 +3,46 @@
   <!-- include macros for robot, end effector, workcell -->
   <xacro:include filename="$(find fanuc_r1000ia_support)/urdf/r1000ia80f_macro.xacro"/>
-  <xacro:include filename="$(find grinding_eef_description)/urdf/grinding_eef_macro.xacro" />
-  <xacro:include filename="$(find ensenso_n10_description)/urdf/ensenso_n10_macro.xacro" />
-  <xacro:include filename="$(find grinding_workcell_description)/urdf/grinding_workcell_macro.xacro" />
+  <xacro:include filename="$(find grinding_eef_description)/urdf/grinding_eef_macro.xacro"/>
+  <xacro:include filename="$(find ensenso_n10_description)/urdf/ensenso_n10_macro.xacro"/>
+  <xacro:include filename="$(find grinding_workcell_description)/urdf/grinding_workcell_macro.xacro"/>
   <!-- create the robot and eef combo itself as a macro -->
   <xacro:macro name="fanuc_r1000ia_ensenso_n10_grinding_support" params="prefix">
-  <!-- instantiate everything -->
-  <xacro:fanuc_r1000ia80f prefix="${prefix}" />
-  <xacro:grinding_eef prefix="${prefix}" />
-  <xacro:ensenso_n10 prefix="${prefix}" />
-  <xacro:grinding_workcell prefix="${prefix}" />
-  <!-- attach workcell to robot model -->
-  <joint name="${prefix}base_link-workcell_frame" type="fixed">
-    <origin xyz="0 0 0" rpy="0 0 0" />
-    <parent link="${prefix}base_link" />
-    <child link="${prefix}grinding_workcell_frame" />
-  </joint>
-  <!-- attach eef to robot model -->
-  <joint name="${prefix}tool0-grinding_eef_frame" type="fixed">
-    <origin xyz="0 0 0" rpy="0 0 0" />
-    <parent link="${prefix}link_6" />
-    <child link="${prefix}grinding_eef_frame" />
-  </joint>
-  <link name="${prefix}grinding_disk_tcp">
+    <!-- instantiate everything -->
+    <xacro:fanuc_r1000ia80f prefix="${prefix}"/>
+    <xacro:grinding_eef prefix="${prefix}"/>
+    <xacro:ensenso_n10 prefix="${prefix}"/>
+    <xacro:grinding_workcell prefix="${prefix}"/>
+    <!-- attach workcell to robot model -->
+    <joint name="${prefix}base_link-workcell_frame" type="fixed">
+      <origin xyz="0 0 0" rpy="0 0 0"/>
+      <parent link="${prefix}base_link"/>
+      <child link="${prefix}grinding_workcell_frame"/>
+    </joint>
+    <!-- attach eef to robot model -->
+    <joint name="${prefix}tool0-grinding_eef_frame" type="fixed">
+      <origin xyz="0 0 0" rpy="0 0 0"/>
+      <parent link="${prefix}link_6"/>
+      <child link="${prefix}grinding_eef_frame"/>
+    </joint>
+    <link name="${prefix}grinding_disk_tcp">
   </link>
-  <joint name="${prefix}tool0-grinding_disk_tcp_frame" type="fixed">
-    <origin xyz="0 0 0.324" rpy="0 0 0" />
-    <parent link="${prefix}tool0" />
-    <child link="${prefix}grinding_disk_tcp" />
-  </joint>
-  <!-- attach Ensenso sensor to robot model (to eef) -->
-  <joint name="${prefix}tool0-ensenso_n10_frame" type="fixed">
-    <origin xyz="-0.215 0.04 0.052" rpy="-1.5707 0 0" />
-    <parent link="${prefix}tool0" />
-    <child link="${prefix}ensenso_n10_frame" />
-  </joint>
-  <link name="${prefix}ensenso_n10_tcp">
+    <joint name="${prefix}tool0-grinding_disk_tcp_frame" type="fixed">
+      <origin xyz="0 0 0.324" rpy="0 0 0"/>
+      <parent link="${prefix}tool0"/>
+      <child link="${prefix}grinding_disk_tcp"/>
+    </joint>
+    <!-- attach Ensenso sensor to robot model (to eef) -->
+    <joint name="${prefix}tool0-ensenso_n10_frame" type="fixed">
+      <origin xyz="-0.215 0.04 0.052" rpy="-1.5707 0 0"/>
+      <parent link="${prefix}tool0"/>
+      <child link="${prefix}ensenso_n10_frame"/>
+    </joint>
+    <link name="${prefix}ensenso_n10_tcp">
   </link>
-  <joint name="${prefix}tool0-ensenso_n10_tcp_frame" type="fixed">
-    <origin xyz="-0.215 0.06 0.052" rpy="-1.5707 0 0" />
-    <parent link="${prefix}tool0" />
-    <child link="${prefix}ensenso_n10_tcp" />
-  </joint>
+    <joint name="${prefix}tool0-ensenso_n10_tcp_frame" type="fixed">
+      <origin xyz="-0.215 0.06 0.052" rpy="-1.5707 0 0"/>
+      <parent link="${prefix}tool0"/>
+      <child link="${prefix}ensenso_n10_tcp"/>
+    </joint>
   </xacro:macro>
 </robot>

File: fanuc_r1000ia_grinding/fanuc_r1000ia_sls_2_grinding_support/urdf/r1000ia_grinding.xacro (robot description, xacro)
@@ -1,4 +1,4 @@
-<?xml version="1.0" ?>
-<robot name="fanuc_r1000ia_grinding" xmlns:xacro="http://ros.org/wiki/xacro">
+<?xml version="1.0"?>
+<robot xmlns:xacro="http://ros.org/wiki/xacro" name="fanuc_r1000ia_grinding">
   <xacro:include filename="$(find fanuc_r1000ia_sls_2_grinding_support)/urdf/r1000ia_grinding_macro.xacro"/>
   <xacro:fanuc_r1000ia_sls_2_grinding_support prefix=""/>

File: fanuc_r1000ia_grinding/fanuc_r1000ia_sls_2_grinding_support/urdf/r1000ia_grinding_macro.xacro (robot description, xacro)
@@ -3,54 +3,54 @@
   <!-- include macros for robot, end effector, workcell -->
   <xacro:include filename="$(find fanuc_r1000ia_support)/urdf/r1000ia80f_macro.xacro"/>
-  <xacro:include filename="$(find grinding_eef_description)/urdf/grinding_eef_macro.xacro" />
+  <xacro:include filename="$(find grinding_eef_description)/urdf/grinding_eef_macro.xacro"/>
   <xacro:include filename="$(find fanuc_r1000ia_sls_2_grinding_support)/urdf/sls_2_interface_macro.xacro"/>
-  <xacro:include filename="$(find sls_2_description)/urdf/sls_2_macro.xacro" />
-  <xacro:include filename="$(find grinding_workcell_description)/urdf/grinding_workcell_macro.xacro" />
+  <xacro:include filename="$(find sls_2_description)/urdf/sls_2_macro.xacro"/>
+  <xacro:include filename="$(find grinding_workcell_description)/urdf/grinding_workcell_macro.xacro"/>
   <!-- create the robot and eef combo itself as a macro -->
   <xacro:macro name="fanuc_r1000ia_sls_2_grinding_support" params="prefix">
-  <!-- instantiate everything -->
-  <xacro:fanuc_r1000ia80f prefix="${prefix}" />
-  <xacro:grinding_eef prefix="${prefix}" />
-  <xacro:sls_2_interface prefix="${prefix}" />
-  <xacro:sls_2 prefix="${prefix}" />
-  <xacro:grinding_workcell prefix="${prefix}" />
-  <!-- attach workcell to robot model -->
-  <joint name="${prefix}base_link-workcell_frame" type="fixed">
-    <origin xyz="0 0 0" rpy="0 0 0" />
-    <parent link="${prefix}base_link" />
-    <child link="${prefix}grinding_workcell_frame" />
-  </joint>
-  <!-- attach eef to robot model -->
-  <joint name="${prefix}tool0-grinding_eef_frame" type="fixed">
-    <origin xyz="0 0 0" rpy="0 0 0" />
-    <parent link="${prefix}link_6" />
-    <child link="${prefix}grinding_eef_frame" />
-  </joint>
-  <link name="${prefix}grinding_disk_tcp">
+    <!-- instantiate everything -->
+    <xacro:fanuc_r1000ia80f prefix="${prefix}"/>
+    <xacro:grinding_eef prefix="${prefix}"/>
+    <xacro:sls_2_interface prefix="${prefix}"/>
+    <xacro:sls_2 prefix="${prefix}"/>
+    <xacro:grinding_workcell prefix="${prefix}"/>
+    <!-- attach workcell to robot model -->
+    <joint name="${prefix}base_link-workcell_frame" type="fixed">
+      <origin xyz="0 0 0" rpy="0 0 0"/>
+      <parent link="${prefix}base_link"/>
+      <child link="${prefix}grinding_workcell_frame"/>
+    </joint>
+    <!-- attach eef to robot model -->
+    <joint name="${prefix}tool0-grinding_eef_frame" type="fixed">
+      <origin xyz="0 0 0" rpy="0 0 0"/>
+      <parent link="${prefix}link_6"/>
+      <child link="${prefix}grinding_eef_frame"/>
+    </joint>
+    <link name="${prefix}grinding_disk_tcp">
   </link>
-  <joint name="${prefix}tool0-grinding_disk_tcp_frame" type="fixed">
-    <origin xyz="0 0 0.324" rpy="0 0 0" />
-    <parent link="${prefix}tool0" />
-    <child link="${prefix}grinding_disk_tcp" />
-  </joint>
-  <!-- attach SLS-2 interface to eef -->
-  <joint name="${prefix}tool0-sls_2_interface_base_link" type="fixed">
-    <origin xyz="-0.267 -0.054 0.0828" rpy="0 0 0" />
-    <parent link="${prefix}tool0" />
-    <child link="${prefix}sls_2_interface_base_link" />
-  </joint>
-  <!-- attach SLS-2 sensor to robot model (to eef) -->
-  <joint name="${prefix}tool0-sls_2_frame" type="fixed">
-    <origin xyz="-0.30 -0.043 0.085" rpy="0 -1.5707 1.5707" />
-    <parent link="${prefix}tool0" />
-    <child link="${prefix}sls_2_frame" />
-  </joint>
-  <link name="${prefix}sls_2_tcp">
+    <joint name="${prefix}tool0-grinding_disk_tcp_frame" type="fixed">
+      <origin xyz="0 0 0.324" rpy="0 0 0"/>
+      <parent link="${prefix}tool0"/>
+      <child link="${prefix}grinding_disk_tcp"/>
+    </joint>
+    <!-- attach SLS-2 interface to eef -->
+    <joint name="${prefix}tool0-sls_2_interface_base_link" type="fixed">
+      <origin xyz="-0.267 -0.054 0.0828" rpy="0 0 0"/>
+      <parent link="${prefix}tool0"/>
+      <child link="${prefix}sls_2_interface_base_link"/>
+    </joint>
+    <!-- attach SLS-2 sensor to robot model (to eef) -->
+    <joint name="${prefix}tool0-sls_2_frame" type="fixed">
+      <origin xyz="-0.30 -0.043 0.085" rpy="0 -1.5707 1.5707"/>
+      <parent link="${prefix}tool0"/>
+      <child link="${prefix}sls_2_frame"/>
+    </joint>
+    <link name="${prefix}sls_2_tcp">
   </link>
-  <joint name="${prefix}tool0-sls_2_tcp_frame" type="fixed">
-    <origin xyz="-0.3 -0.1 0.06" rpy="1.5707 0 0" />
-    <parent link="${prefix}tool0" />
-    <child link="${prefix}sls_2_tcp" />
-  </joint>
+    <joint name="${prefix}tool0-sls_2_tcp_frame" type="fixed">
+      <origin xyz="-0.3 -0.1 0.06" rpy="1.5707 0 0"/>
+      <parent link="${prefix}tool0"/>
+      <child link="${prefix}sls_2_tcp"/>
+    </joint>
   </xacro:macro>
 </robot>

File: fanuc_r1000ia_grinding/fanuc_r1000ia_sls_2_grinding_support/urdf/sls_2_interface.xacro (robot description, xacro)
@@ -1,4 +1,4 @@
-<?xml version="1.0" ?>
-<robot name="sls_2_interface" xmlns:xacro="http://ros.org/wiki/xacro">
+<?xml version="1.0"?>
+<robot xmlns:xacro="http://ros.org/wiki/xacro" name="sls_2_interface">
   <xacro:include filename="$(find fanuc_r1000ia_sls_2_grinding_support)/urdf/sls_2_interface_macro.xacro"/>
   <xacro:sls_2_interface prefix=""/>

File: fanuc_r1000ia_grinding/grinding_effector_description/urdf/grinding_eef.xacro (robot description, xacro)
@@ -1,4 +1,4 @@
-<?xml version="1.0" ?>
-<robot name="grinding_eef" xmlns:xacro="http://ros.org/wiki/xacro">
+<?xml version="1.0"?>
+<robot xmlns:xacro="http://ros.org/wiki/xacro" name="grinding_eef">
   <xacro:include filename="$(find grinding_eef_description)/urdf/grinding_eef_macro.xacro"/>
   <xacro:grinding_eef prefix=""/>

File: fanuc_r1000ia_grinding/grinding_workcell_description/urdf/grinding_workcell.xacro (robot description, xacro)
@@ -1,4 +1,4 @@
-<?xml version="1.0" ?>
-<robot name="grinding_workcell" xmlns:xacro="http://ros.org/wiki/xacro">
+<?xml version="1.0"?>
+<robot xmlns:xacro="http://ros.org/wiki/xacro" name="grinding_workcell">
   <xacro:include filename="$(find grinding_workcell_description)/urdf/grinding_workcell_macro.xacro"/>
   <xacro:grinding_workcell prefix=""/>

File: sensors/ensenso_n10_description/urdf/ensenso_n10.xacro (robot description, xacro)
@@ -1,4 +1,4 @@
-<?xml version="1.0" ?>
-<robot name="ensenso_n10" xmlns:xacro="http://ros.org/wiki/xacro">
+<?xml version="1.0"?>
+<robot xmlns:xacro="http://ros.org/wiki/xacro" name="ensenso_n10">
   <xacro:include filename="$(find ensenso_n10_description)/urdf/ensenso_n10_macro.xacro"/>
   <xacro:ensenso_n10 prefix=""/>

File: sensors/kinect_v1_description/urdf/kinect_v1.xacro (robot description, xacro)
@@ -1,4 +1,4 @@
-<?xml version="1.0" ?>
-<robot name="kinect_v1" xmlns:xacro="http://ros.org/wiki/xacro">
+<?xml version="1.0"?>
+<robot xmlns:xacro="http://ros.org/wiki/xacro" name="kinect_v1">
   <xacro:include filename="$(find kinect_v1_description)/urdf/kinect_v1_macro.xacro"/>
   <xacro:kinect_v1 prefix=""/>

File: sensors/sls_2_description/urdf/sls_2.xacro (robot description, xacro)
@@ -1,4 +1,4 @@
-<?xml version="1.0" ?>
-<robot name="sls_2" xmlns:xacro="http://ros.org/wiki/xacro">
+<?xml version="1.0"?>
+<robot xmlns:xacro="http://ros.org/wiki/xacro" name="sls_2">
   <xacro:include filename="$(find sls_2_description)/urdf/sls_2_macro.xacro"/>
   <xacro:sls_2 prefix=""/>
