Commit message: Use xmlindent to fix indentation

File: fanuc_m10ia_ensenso/fanuc_m10ia_ensenso_support/urdf/m10ia_ensenso_eef_macro.xacro (robot description, xacro)
@@ -24,5 +24,5 @@
     </joint>
     <link name="${prefix}ensenso_tcp">
-  </link>
+    </link>
     <joint name="${prefix}tool0-ensenso_tcp_frame" type="fixed">
       <origin xyz="0 -0.088 0.035" rpy="0 0 -1.5707"/>

File: sensors/sls_2_description/urdf/sls_2_macro.xacro (robot description, xacro)
@@ -61,5 +61,5 @@
       <origin xyz="0 0 0" rpy="0 0 0"/>
     </joint>
-   <joint name="${prefix}sls_2_camera_inter_cam" type="fixed">
+    <joint name="${prefix}sls_2_camera_inter_cam" type="fixed">
       <parent link="${prefix}sls_2_camera" />
       <child link="${prefix}sls_2_inter_cam" />
