Commit message: Improve xacro formatting

File: fanuc_m10ia_kinect/fanuc_m10ia_kinect_support/urdf/m10ia_kinect_eef_macro.xacro (robot description, xacro)
@@ -23,6 +23,5 @@
       <child link="${prefix}kinect_v1_frame"/>
     </joint>
-    <link name="${prefix}kinect_tcp">
-  </link>
+    <link name="${prefix}kinect_tcp"/>
     <joint name="${prefix}tool0-kinect_tcp_frame" type="fixed">
       <origin xyz="0 -0.01 0.028" rpy="0 0 0"/>

File: fanuc_r1000ia_grinding/fanuc_r1000ia_ensenso_n10_grinding_support/urdf/r1000ia_grinding_macro.xacro (robot description, xacro)
@@ -25,6 +25,5 @@
       <child link="${prefix}grinding_eef_frame"/>
     </joint>
-    <link name="${prefix}grinding_disk_tcp">
-  </link>
+    <link name="${prefix}grinding_disk_tcp"/>
     <joint name="${prefix}tool0-grinding_disk_tcp_frame" type="fixed">
       <origin xyz="0 0 0.324" rpy="0 0 0"/>
@@ -38,6 +37,5 @@
       <child link="${prefix}ensenso_n10_frame"/>
     </joint>
-    <link name="${prefix}ensenso_n10_tcp">
-  </link>
+    <link name="${prefix}ensenso_n10_tcp"/>
     <joint name="${prefix}tool0-ensenso_n10_tcp_frame" type="fixed">
       <origin xyz="-0.215 0.06 0.052" rpy="-1.5707 0 0"/>

File: fanuc_r1000ia_grinding/fanuc_r1000ia_sls_2_grinding_support/urdf/r1000ia_grinding_macro.xacro (robot description, xacro)
@@ -27,6 +27,5 @@
       <child link="${prefix}grinding_eef_frame"/>
     </joint>
-    <link name="${prefix}grinding_disk_tcp">
-  </link>
+    <link name="${prefix}grinding_disk_tcp"/>
     <joint name="${prefix}tool0-grinding_disk_tcp_frame" type="fixed">
       <origin xyz="0 0 0.324" rpy="0 0 0"/>
@@ -46,6 +45,5 @@
       <child link="${prefix}sls_2_frame"/>
     </joint>
-    <link name="${prefix}sls_2_tcp">
-  </link>
+    <link name="${prefix}sls_2_tcp"/>
     <joint name="${prefix}tool0-sls_2_tcp_frame" type="fixed">
       <origin xyz="-0.3 -0.1 0.06" rpy="1.5707 0 0"/>
