Commit message: Deprecate old work-cell and add new as default

File: fanuc_r1000ia_grinding/grinding_workcell_description/urdf/grinding_old_workcell_macro.xacro (robot description, xacro)
@@ -4,7 +4,7 @@
     <link name="${prefix}grinding_workcell_frame">
       <visual>
-        <origin xyz="0 0 -0.52" rpy="0 0 0"/>
+        <origin xyz="0 0 0" rpy="0 0 0"/>
         <geometry>
-          <mesh filename="package://grinding_workcell_description/meshes/visual/grinding_workcell.dae"/>
+          <mesh filename="package://grinding_workcell_description/meshes/visual/grinding_old_workcell.dae"/>
         </geometry>
         <material name="light-grey">
@@ -13,7 +13,7 @@
       </visual>
       <collision>
-        <origin xyz="0 0 -0.52" rpy="0 0 0"/>
+        <origin xyz="0 0 0" rpy="0 0 0"/>
         <geometry>
-          <mesh filename="package://grinding_workcell_description/meshes/collision/grinding_workcell.stl"/>
+          <mesh filename="package://grinding_workcell_description/meshes/collision/grinding_old_workcell.stl"/>
         </geometry>
       </collision>
