Commit message: Tweak Fanuc with SLS-2 to use new SLS-2 description

File: fanuc_r1000ia_grinding/fanuc_r1000ia_sls_2_grinding_support/urdf/r1000ia_grinding_macro.xacro (robot description, xacro)
@@ -14,5 +14,5 @@
     <xacro:grinding_eef prefix="${prefix}"/>
     <xacro:sls_2_interface prefix="${prefix}"/>
-    <xacro:sls_2 prefix="${prefix}"/>
+    <xacro:sls_2 prefix="${prefix}" camera_angle="-0.349" camera_trans="-0.18"/>
     <!-- attach workcell to robot model -->
     <joint name="${prefix}base_link-workcell_frame" type="fixed">
@@ -41,5 +41,5 @@
     <!-- attach SLS-2 sensor to robot model (to eef) -->
     <joint name="${prefix}tool0-sls_2_frame" type="fixed">
-      <origin xyz="-0.30 -0.043 0.085" rpy="0 -1.5707 1.5707"/>
+      <origin xyz="-0.35 -0.056 0.072" rpy="0.349 -1.5707 1.5707"/>
       <parent link="${prefix}tool0"/>
       <child link="${prefix}sls_2_frame"/>

Commit message: Add extrinsic calibration package

File: fanuc_r1000ia_grinding/fanuc_r1000ia_sls_2_grinding_support/urdf/r1000ia_grinding_macro.xacro (robot description, xacro)
@@ -1,4 +1,6 @@
 <?xml version="1.0"?>
 <robot xmlns:xacro="http://ros.org/wiki/xacro">
+  <!-- Macro to create 6 joints/links between tool0 and SLS-2 frame -->
+  <xacro:include filename="$(find industrial_extrinsic_cal)/urdf/calibration_transform_macro.xacro"/>
   <!-- include macros for robot, end effector, workcell -->
   <xacro:include filename="$(find grinding_workcell_description)/urdf/grinding_workcell_macro.xacro"/>
@@ -14,5 +16,5 @@
     <xacro:grinding_eef prefix="${prefix}"/>
     <xacro:sls_2_interface prefix="${prefix}"/>
-    <xacro:sls_2 prefix="${prefix}" camera_angle="-0.349" camera_trans="-0.18"/>
+    <xacro:sls_2 prefix="${prefix}" camera_angle="-0.2792" camera_trans="0.2"/>
     <!-- attach workcell to robot model -->
     <joint name="${prefix}base_link-workcell_frame" type="fixed">
@@ -39,16 +41,10 @@
       <child link="${prefix}sls_2_interface_base_link"/>
     </joint>
-    <!-- attach SLS-2 sensor to robot model (to eef) -->
-    <joint name="${prefix}tool0-sls_2_frame" type="fixed">
-      <origin xyz="-0.35 -0.056 0.072" rpy="0.349 -1.5707 1.5707"/>
-      <parent link="${prefix}tool0"/>
-      <child link="${prefix}sls_2_frame"/>
-    </joint>
-    <link name="${prefix}sls_2_tcp"/>
-    <joint name="${prefix}tool0-sls_2_tcp_frame" type="fixed">
-      <origin xyz="-0.3 -0.1 0.06" rpy="1.5707 0 0"/>
-      <parent link="${prefix}tool0"/>
-      <child link="${prefix}sls_2_tcp"/>
-    </joint>
+    <!-- Create 5 links and 6 joints between link sls_2_frame and tool0 link
+         Uses child link as the child link of the 6th joint -->
+    <xacro:calibration_definitions child_link="${prefix}sls_2_frame" parent_link="${prefix}tool0" />
+    <!-- Calibration target definitions -->
+    <link name="target_frame"/>
+    <xacro:calibration_definitions child_link="target_frame" parent_link="base"/>
   </xacro:macro>
 </robot>

Commit message: Modify localisation of grinding disk origin

File: fanuc_r1000ia_grinding/fanuc_r1000ia_sls_2_grinding_support/urdf/r1000ia_grinding_macro.xacro (robot description, xacro)
@@ -29,5 +29,5 @@
     <link name="${prefix}grinding_disk_tcp"/>
     <joint name="${prefix}tool0-grinding_disk_tcp_frame" type="fixed">
-      <origin xyz="0 0 0.324" rpy="0 0 0"/>
+      <origin xyz="0 0 0.327" rpy="0 0 0"/>
       <parent link="${prefix}tool0"/>
       <child link="${prefix}grinding_disk_tcp"/>
